Commit message: change joint type

File: src/arm_description/urdf/arm.urdf.xacro (robot description, xacro)
@@ -65,5 +65,45 @@
   <!-- Generates child joint of parent -->
   <xacro:macro name="arm_joint" params="child parent dist:=0 axis">
-    <joint name="${parent}_${child}_joint" type="revolute">
+    <joint name="${parent}_${child}_joint" type="prismatic">
+      <origin xyz="0 0 ${dist}" rpy="0 0 0"/>
+      <parent link="${parent}"/>
+      <child link="${child}"/>
+      <axis xyz="${axis}"/>
+      <limit effort="40.0"
+             velocity="1.0"
+             lower="${-PI}"
+             upper="${PI}"/>
+    </joint>
+    <!-- Required for ROS control -->
+    <transmission name="${parent}_${child}_transmission">
+      <type>transmission_interface/SimpleTransmission</type>
+      <joint name="${parent}_${child}_joint">
+        <hardwareInterface>hardware_interface/EffortJointInterface</hardwareInterface>
+      </joint>
+      <actuator name="${parent}_${child}_actuator"/>
+    </transmission>
+    <link name="${parent}">
+      <xacro:prism_vci length="${dist}" side="${link_side}">
+        <origin xyz="0 0 ${dist/2}" rpy="0 0 0"/>
+      </xacro:prism_vci>
+      <xacro:cylinder_vc radius="${joint_radius}" length="${joint_length}">
+        <xacro:if value="${axis=='0 0 1'}">
+          <origin xyz="0 0 ${dist}" rpy="0 0 0"/>
+        </xacro:if>
+        <xacro:if value="${axis=='1 0 0'}">
+          <origin xyz="0 0 ${dist}" rpy="0 ${PI/2} 0"/>
+        </xacro:if>
+        <xacro:if value="${axis=='0 1 0'}">
+          <origin xyz="0 0 ${dist}" rpy="${PI/2} 0 0"/>
+        </xacro:if>
+      </xacro:cylinder_vc>
+    </link>
+    <gazebo reference="${parent}">
+      <material>Gazebo/Orange</material>
+    </gazebo>
+  </xacro:macro>
+  <!-- Generates child joint of parent -->
+  <xacro:macro name="arm_joint_fix" params="child parent dist:=0 axis">
+    <joint name="${parent}_${child}_joint" type="fixed">
       <origin xyz="0 0 ${dist}" rpy="0 0 0"/>
       <parent link="${parent}"/>

Commit message: add new xacro:macro "arm_joint_fix"

File: src/arm_description/urdf/arm.urdf.xacro (robot description, xacro)
@@ -65,5 +65,5 @@
   <!-- Generates child joint of parent -->
   <xacro:macro name="arm_joint" params="child parent dist:=0 axis">
-    <joint name="${parent}_${child}_joint" type="prismatic">
+    <joint name="${parent}_${child}_joint" type="revolute">
       <origin xyz="0 0 ${dist}" rpy="0 0 0"/>
       <parent link="${parent}"/>
